File: images/FPGA_HD44780_Hello.sch (KiCad schematic (older format))
At the start: 4 parts, among them U2 74HCT541, U3 LCD-016N002L

Commit message: test circuit schematic
Parts:
- added D0, D1, D2, D3: LED, symbol Device:LED
- added R1, R2, R3, R4: 1K, symbol Device:R_Small_US
- added SW1: SW_Push, symbol Switch:SW_Push
- gave numbers to parts that had none: 1
Connections:
- net +5V: now also U1.~ (J8/OSC_OUT), U2.20 (VCC)
- net GND: now also U1.~ (J8/OSC_OUT), SW1.1
- net at U2.2 (A0): now also U1.34 (DPIO-(37))
- net at U2.3 (A1): now also U1.37 (GBIN/DPIO+(34))
- net at U2.4 (A2): now also U1.43 (DPIO+(36))
- net at U2.5 (A3): now also U1.23 (DPIO+(25))
- net at U2.6 (A4): now also U1.25 (DPIO-(23))
- net at U2.7 (A5): now also U1.26 (DPIO+(27))
- net at U2.8 (A6): now also U1.27 (DPIO-(26))
- net at U1.28 (PIO): now also D3.1 (K)
- net at U1.36 (DPIO-(43)): now also D0.1 (K)
- net at U1.38 (DPIO-(42)): now also D2.1 (K)
- net at U1.42 (DPIO+(38)): now also D1.1 (K)
- net at U1.44 (DPIO-(47)): now also SW1.2
- new net: D3.2 (A), R1.2
- new net: D2.2 (A), R2.2
- new net: D1.2 (A), R3.2
- new net: D0.2 (A), R4.2
- new net +3V3: R1.1, R2.1, R3.1, R4.1, U1.~ (J8/OSC_OUT)
Other:
- moved on the sheet: RV1, U1, U2, U3
